File: circuitDesign/circuitDesign.sch (KiCad schematic (older format))
At the start: 11 parts, among them IC1 ATTINY25-P, X1 CRYSTAL 20MHz

Commit message: Added diode values
Parts:
- D1: value ZENER -> ZENER 1N4733
- R1: value R -> R 220
Changed lines of the file:
@@
 P 8200 3850
 F 0 "D1" H 8200 3950 50  0000 C CNN
-F 1 "ZENER" H 8200 3750 40  0000 C CNN
+F 1 "ZENER 1N4733" H 8200 3750 40  0000 C CNN
 F 2 "~" H 8200 3850 60  0000 C CNN
 F 3 "~" H 8200 3850 60  0000 C CNN
@@
 P 8200 2700
 F 0 "R1" V 8280 2700 40  0000 C CNN
-F 1 "R" V 8207 2701 40  0000 C CNN
+F 1 "R 220" V 8207 2701 40  0000 C CNN
 F 2 "~" V 8130 2700 30  0000 C CNN
 F 3 "~" H 8200 2700 30  0000 C CNN
