File: circuitDesign/transponder/transponder.kicad_pcb (KiCad board)
At the start: 2 copper layers, 45.7 x 45.7 mm, 13 parts, among them IC1 ATTINY85-P, P1 CONN_2, X1 CRYSTAL

Commit message: PCB work, and more
Parts:
- removed D2: ZENER, SM2010
- removed R3: 75, SM0805
- added U1: L78L05_SOT89, TO_SOT_Packages_SMD:SOT-89-3, F.Cu at (110.2, 104.9)
- C1, C2, C3: footprint SM0805 -> Capacitors_SMD:C_0805
- C4: footprint SM1206 -> Capacitors_Tantalum_SMD:CP_Tantalum_Case-A_EIA-3216-18_Reflow
- D1: footprint LED-0805 -> LEDs:LED_0805
- D3: footprint SM0805 -> Diodes_SMD:D_0805
- IC1: footprint SO8_200mil_wide -> Housings_DIP:DIP-8_W7.62mm_Socket
- P1: footprint PIN_ARRAY_2X1 -> Connectors:PINHEAD1-2
- R1, R2: footprint SM0805 -> Resistors_SMD:R_0805
- X1: footprint CRYSTAL-NX5032GA -> Crystals:Crystal_SMD_5032-2pin_5.0x3.2mm
- moved P1 76.2 mm to (102.4, 104.4), turned to 180 degrees
- moved IC1 74.0 mm to (103.9, 109.0), turned to 0 degrees
- moved C1 71.3 mm to (99.1, 109.5)
- moved D3 69.4 mm to (105.7, 103.4), turned to 180 degrees
- moved X1 66.1 mm to (99.3, 115.3)
- moved D1 65.9 mm to (114.0, 106.2), turned to 90 degrees
- moved C3 65.4 mm to (102.9, 119.1), turned to 0 degrees
- moved R2 65.0 mm to (114.0, 111.3), turned to 270 degrees
- moved C2 64.9 mm to (113.3, 119.9), turned to 0 degrees
- moved R1 62.9 mm to (114.0, 115.8), turned to 90 degrees
- moved C4 62.7 mm to (107.7, 119.4), turned to 180 degrees
Connections:
- C4 pad 1: N-0000011 -> Net-(C4-Pad1)
- D1 pad 2: GND -> Net-(C4-Pad1)
- D3 pad 1: +BATT -> Net-(D3-Pad1)
- IC1 pad 1: N-0000011 -> (no net)
- IC1 pad 8: N-0000011 -> Net-(C4-Pad1)
Routing:
- net (no net): track 0.00 -> 247.3 mm
- net GND: track 0.00 -> 32.8 mm
- net N-0000011: track 23.0 -> 0.00 mm
- net Net-(C4-Pad1): track 0.00 -> 17.3 mm
- net Net-(IC1-Pad6): track 8.45 -> 3.43 mm
- net Net-(IC1-Pad7): track 6.05 -> 2.16 mm
- net Net-(C1-Pad1): track 11.1 -> 8.41 mm
- net Net-(D1-Pad1): track 2.12 -> 0.00 mm
- net Net-(D3-Pad1): track 0.00 -> 2.05 mm
- net +BATT: track 1.65 -> 0.00 mm
- net Net-(C2-Pad2): track 1.65 -> 3.28 mm
- net Net-(C2-Pad1): track 2.43 -> 3.68 mm
- net Net-(C3-Pad1): track 10.7 -> 9.94 mm
- removed copper zone on F.Cu, net GND
Other:
- board size 45.7 x 45.7 mm -> 22.9 x 22.9 mm
- net class pcb test added: clearance 0.127, trace_width 0.127, via_dia 0.889, via_drill 0.635
- rule trace_min: 0.254 -> 0.127
